File: basic_macropad.kicad_pcb (KiCad board)
At the start: 2 copper layers, 92.9 x 50.8 mm, 38 parts, among them SW1 SW_Push, SW2 Rotary_Encoder_Switch, U1 ATmega32U4-AU, U2 PRTR5V0U2X, Y1 16MHz

Commit message: Final
Parts:
- removed R7: 500, Resistor_SMD:R_0805_2012Metric
- added H5: MountingHole_Pad, MountingHole:MountingHole_2.2mm_M2_Pad, F.Cu at (146.1, 122.2)
- added H6: MountingHole_Pad, MountingHole:MountingHole_2.2mm_M2_Pad, F.Cu at (232.6, 122.2)
- added H7: MountingHole_Pad, MountingHole:MountingHole_2.2mm_M2_Pad, F.Cu at (146.1, 166.7)
- added H8: MountingHole_Pad, MountingHole:MountingHole_2.2mm_M2_Pad, F.Cu at (232.6, 166.7)
- added LOGO: , Logos:LOGO_Smallest, F.Cu at (153.0, 83.2)
- added REF**: breakaway-mousebites, random-keyboard-parts:breakaway-mousebites, F.Cu at (212.7, 119.0)
- added REF**: breakaway-mousebites, random-keyboard-parts:breakaway-mousebites, F.Cu at (212.7, 115.2)
- added REF**: breakaway-mousebites, random-keyboard-parts:breakaway-mousebites, F.Cu at (165.9, 119.0)
- added REF**: breakaway-mousebites, random-keyboard-parts:breakaway-mousebites, F.Cu at (165.9, 115.2)
- H1, H2, H3, H4: value MountingHole -> MountingHole_Pad; footprint MountingHole:MountingHole_2.2mm_M2 -> MountingHole:MountingHole_2.2mm_M2_Pad
- moved R4 37.0 mm to (176.2, 69.8)
- moved D6 10.5 mm to (226.2, 75.4)
- moved D2 6.64 mm to (208.8, 80.2)
- moved D1 6.46 mm to (189.7, 80.2)
- moved D3 6.46 mm to (189.7, 99.2)
- moved D4 6.46 mm to (208.8, 99.2)
- moved D5 6.46 mm to (227.8, 99.2)
- moved D7 0.76 mm to (173.8, 88.1), turned to 0 degrees
- turned D8 to 180 degrees
Connections:
- D7 pad 4: Net-(D7-Pad4) -> RGBLED
- H1 pad 1: (no net) -> Net-(H1-Pad1)
- H2 pad 1: (no net) -> Net-(H2-Pad1)
- H3 pad 1: (no net) -> Net-(H3-Pad1)
- H4 pad 1: (no net) -> Net-(H4-Pad1)
Routing:
- net GND: track 200.7 -> 277.6 mm, vias 2 -> 4
- net +5V: track 120.8 -> 177.5 mm, vias 7 -> 6
- net Net-(D6-Pad2): track 16.4 -> 3.75 mm
- net Net-(D7-Pad2): track 29.5 -> 39.1 mm
- net RGBLED: track 9.33 -> 18.2 mm
- net Net-(D7-Pad4): track 7.06 -> 0.00 mm
- net Net-(D2-Pad2): track 11.2 -> 4.16 mm
- net Net-(D5-Pad2): track 10.3 -> 4.16 mm
- net Net-(D4-Pad2): track 10.3 -> 4.16 mm
- net Net-(D3-Pad2): track 10.3 -> 4.16 mm
- net Net-(D1-Pad2): track 10.3 -> 4.16 mm
- net ROW0: track 71.6 -> 76.9 mm, vias 4 -> 2
- net ENC_B: track 99.7 -> 97.8 mm, vias 2 -> 0
- net ENC_A: track 103.4 -> 101.8 mm, vias 2 -> 0
- net ROW1: track 69.0 -> 68.4 mm
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- added copper zone on B.Cu, net GND
Other:
- board size 92.9 x 50.8 mm -> 92.9 x 105.6 mm
- board text added: "prototype designed by tristan colby"
- board text added: "trco.dev"
