File: basic_macropad.sch (KiCad schematic (older format))
At the start: 24 parts, among them SW1 SW_Push, U1 ATmega32U4-AU, Y1 16MHz

Commit message: Almost done
Parts:
- removed USB1: Molex-0548190589, random-keyboard-parts:Molex-0548190589, symbol random-keyboard-parts:Molex-0548190589
- added D5, D6: SOD-123, Diode_SMD:D_SOD-123, symbol Device:D_Small
- added D7, D8: WS2812B, LED_SMD:LED_WS2812B_PLCC4_5.0x5.0mm_P3.2mm, symbol LED:WS2812B
- added H1, H2, H3, H4: MountingHole, MountingHole:MountingHole_2.2mm_M2, symbol Mechanical:MountingHole
- added MX5: MX-NoLED, MX_Only:MXOnly-1U-Hotswap, symbol MX_Alps_Hybrid:MX-NoLED
- added R5, R6: 22, Resistor_SMD:R_0805_2012Metric, symbol Device:R_Small
- added R7: 500, Resistor_SMD:R_0805_2012Metric, symbol Device:R_Small
- added SW2: Rotary_Encoder_Switch, Rotary_Encoder:RotaryEncoder_Alps_EC11E-Switch_Vertical_H20mm_CircularMountingHoles, symbol Device:Rotary_Encoder_Switch
- added U2: PRTR5V0U2X, random-keyboard-parts:SOT143B, symbol random-keyboard-parts:PRTR5V0U2X
- added USB1: HRO-TYPE-C-31-M-12, Type-C:HRO-TYPE-C-31-M-12-Assembly, symbol Type-C:HRO-TYPE-C-31-M-12
- C2: value 22pF -> 0.1uF
- C3: value C_Small -> 0.1uF
- C4: value 0.1uF -> 10uF
- C5: value 0.1uF -> 22pF
- C6: value 1uF -> 22pF
- C7: value 10uF -> 1uF
- F1: value Polyfuse_Small -> 500mA; footprint Diode_SMD:D_1206_3216Metric -> Fuse:Fuse_1206_3216Metric
- MX1, MX2, MX3, MX4: footprint MX_Alps_Hybrid:MX-1U-NoLED -> MX_Only:MXOnly-1U-Hotswap
- R1: value 22 -> 10k
- R2: value 22 -> 5.1k
- R3: value 10k -> 5.1k
Connections:
- net +5V: now also C2.1, C3.1, R4.1, U1.24 (AVCC), U1.44 (AVCC), D7.1 (VDD), D8.1 (VDD); no longer C5.1, C7.1, R3.1
- net COL0: now also MX3.1 (COL), U1.27 (PD7); no longer MX2.1 (COL)
- net COL1: now also MX2.1 (COL), U1.29 (PB5); no longer MX3.1 (COL)
- net D+: now also U1.4 (D+), R6.2; no longer R2.2
- net D-: now also U1.3 (D-), R5.2; no longer R1.2
- net GND: now also C6.2, R1.1, R2.2, R3.2, U1.15 (GND), U1.23 (GND), U1.35 (GND), U1.43 (GND), D7.3 (VSS), D8.3 (VSS), SW2.C, U2.1 (GND), USB1.1 (GND), USB1.12 (GND), USB1.13 (SHIELD); no longer C6.1, R4.1
- net ROW0: now also D2.1 (K), U1.26 (PD6), D6.1 (K); no longer D3.1 (K)
- net ROW1: now also D3.1 (K), U1.28 (PB4), D5.1 (K); no longer D2.1 (K)
- net VCC: now also U2.4 (VCC), USB1.11 (VBUS), USB1.2 (VBUS)
- net at SW1.2, U1.13 (~RESET): now also R4.2; no longer R3.2
- net at U1.16 (XTAL2), Y1.3: now also C6.1; no longer C3.1
- net at U1.17 (XTAL1), Y1.1: now also C5.1; no longer C2.1
- net RGBLED: now reaches U1.25 (PD4)
- net RGBLED: now also R7.2
- net COL2: now reaches U1.30 (PB6)
- net COL2: now also MX5.1 (COL), SW2.S2
- net ENC_A: now reaches U1.31 (PC6)
- net ENC_A: now also SW2.A
- net ENC_B: now reaches U1.32 (PC7)
- net ENC_B: now also SW2.B
- net at U1.33 (~HWB~/PE2): now also R1.2; no longer R4.2
- net at R2.1: now also USB1.10 (CC2); no longer U1.4 (D+)
- net at U1.6 (UCAP): now also C7.1; no longer C6.2
- new net: R3.1, USB1.4 (CC1)
- new net: R5.1, U2.3 (IO2), USB1.5 (DN2), USB1.7 (DN1)
- new net: R6.1, U2.2 (IO1), USB1.6 (DP1), USB1.8 (DP2)
- new net: D6.2 (A), SW2.S1
- new net: D5.2 (A), MX5.2 (ROW)
- new net: D7.2 (DOUT), D8.4 (DIN)
- new net: D7.4 (DIN), R7.1
- no-connect marks 0 -> 3

Commit message: Final
Parts:
- removed H1, H2, H3, H4: MountingHole, MountingHole:MountingHole_2.2mm_M2, symbol Mechanical:MountingHole
- removed R7: 500, Resistor_SMD:R_0805_2012Metric, symbol Device:R_Small
- added H1, H2, H3, H4: MountingHole_Pad, MountingHole:MountingHole_2.2mm_M2_Pad, symbol Mechanical:MountingHole_Pad
- C1, C2, C3: LCSC (none) -> C49678
- C4: LCSC (none) -> C15850
- C5, C6: LCSC (none) -> C1804
- C7: LCSC (none) -> C28323
- D1, D2, D3, D4, D5, D6: LCSC (none) -> C8598
- D7, D8: LCSC (none) -> C114586
- F1: LCSC (none) -> C206993
- R1, R4: LCSC (none) -> C17414
- R2, R3: LCSC (none) -> C27834
- R5, R6: LCSC (none) -> C17561
- SW1: LCSC (none) -> C318884
- U1: LCSC (none) -> C44854
- Y1: LCSC (none) -> C13738
Connections:
- net RGBLED: now also D7.4 (DIN)
- no-connect marks 3 -> 21
Changed lines of the file:
@@
 F 2 "Package_QFP:TQFP-44_10x10mm_P0.8mm" H 3900 3040 50  0001 C CIN
 F 3 "http://ww1.microchip.com/downloads/en/DeviceDoc/Atmel-7766-8-bit-AVR-ATmega16U4-32U4_Datasheet.pdf" H 3900 3040 50  0001 C CNN
+F 4 "C44854" H 3900 3040 50  0001 C CNN "LCSC"
 	1    3900 3040
 	1    0    0    -1
@@
 F 2 "Resistor_SMD:R_0805_2012Metric" H 5580 3640 50  0001 C CNN
 F 3 "~" H 5580 3640 50  0001 C CNN
+F 4 "C17414" V 5580 3640 50  0001 C CNN "LCSC"
 	1    5580 3640
 	0    1    1    0
@@
 F 2 "Capacitor_SMD:C_0805_2012Metric" H 2720 2940 50  0001 C CNN
 F 3 "~" H 2720 2940 50  0001 C CNN
+F 4 "C28323" H 2720 2940 50  0001 C CNN "LCSC"
 	1    2720 2940
 	1    0    0    -1
@@
 F 2 "Capacitor_SMD:C_0805_2012Metric" H 710 3890 50  0001 C CNN
 F 3 "~" H 710 3890 50  0001 C CNN
+F 4 "C49678" H 710 3890 50  0001 C CNN "LCSC"
 	1    710  3890
 	1    0    0    -1
@@
 F 2 "Capacitor_SMD:C_0805_2012Metric" H 980 3890 50  0001 C CNN
 F 3 "~" H 980 3890 50  0001 C CNN
+F 4 "C49678" H 980 3890 50  0001 C CNN "LCSC"
 	1    980  3890
 	1    0    0    -1
@@
 F 2 "Capacitor_SMD:C_0805_2012Metric" H 1250 3890 50  0001 C CNN
 F 3 "~" H 1250 3890 50  0001 C CNN
+F 4 "C49678" H 1250 3890 50  0001 C CNN "LCSC"
 	1    1250 3890
 	1    0    0    -1
@@
 F 2 "Capacitor_SMD:C_0805_2012Metric" H 1520 3890 50  0001 C CNN
 F 3 "~" H 1520 3890 50  0001 C CNN
+F 4 "C15850" H 1520 3890 50  0001 C CNN "LCSC"
 	1    1520 3890
 	1    0    0    -1
@@
 F 2 "Capacitor_SMD:C_0805_2012Metric" H 1810 1670 50  0001 C CNN
 F 3 "~" H 1810 1670 50  0001 C CNN
+F 4 "C1804" V 1810 1670 50  0001 C CNN "LCSC"
 	1    1810 1670
 	0    1    1    0
@@
 F 2 "Capacitor_SMD:C_0805_2012Metric" H 1810 2010 50  0001 C CNN
 F 3 "~" H 1810 2010 50  0001 C CNN
+F 4 "C1804" V 1810 2010 50  0001 C CNN "LCSC"
 	1    1810 2010
 	0    1    1    0
@@
 F 2 "Crystal:Crystal_SMD_3225-4Pin_3.2x2.5mm" H 2130 1840 50  0001 C CNN
 F 3 "~" H 2130 1840 50  0001 C CNN
+F 4 "C13738" V 2130 1840 50  0001 C CNN "LCSC"
 	1    2130 1840
 	0    1    1    0
@@
 F 2 "random-keyboard-parts:SKQG-1155865" H 2730 1740 50  0001 C CNN
 F 3 "~" H 2730 1740 50  0001 C CNN
+F 4 "C318884" H 2730 1540 50  0001 C CNN "LCSC"
 	1    2730 1540
 	1    0    0    -1
@@
 F 2 "Resistor_SMD:R_0805_2012Metric" H 3110 1290 50  0001 C CNN
 F 3 "~" H 3110 1290 50  0001 C CNN
+F 4 "C17414" H 3110 1290 50  0001 C CNN "LCSC"
 	1    3110 1290
 	1    0    0    -1
@@
 F 2 "Diode_SMD:D_SOD-123" V 6960 2350 50  0001 C CNN
 F 3 "~" V 6960 2350 50  0001 C CNN
+F 4 "C8598" V 6960 2350 50  0001 C CNN "LCSC"
 	1    6960 2350
 	0    -1   -1   0
@@
 F 2 "Diode_SMD:D_SOD-123" V 7640 2350 50  0001 C CNN
 F 3 "~" V 7640 2350 50  0001 C CNN
+F 4 "C8598" V 7640 2350 50  0001 C CNN "LCSC"
 	1    7640 2350
 	0    -1   -1   0
@@
 F 2 "Diode_SMD:D_SOD-123" V 6960 3000 50  0001 C CNN
 F 3 "~" V 6960 3000 50  0001 C CNN
+F 4 "C8598" V 6960 3000 50  0001 C CNN "LCSC"
 	1    6960 3000
 	0    -1   -1   0
@@
 F 2 "Diode_SMD:D_SOD-123" V 7640 3000 50  0001 C CNN
 F 3 "~" V 7640 3000 50  0001 C CNN
+F 4 "C8598" V 7640 3000 50  0001 C CNN "LCSC"
 	1    7640 3000
 	0    -1   -1   0
@@
 F 2 "Fuse:Fuse_1206_3216Metric" H 2780 5575 50  0001 L CNN
 F 3 "~" H 2730 5775 50  0001 C CNN
+F 4 "C206993" V 2730 5775 50  0001 C CNN "LCSC"
 	1    2730 5775
 	0    1    1    0
@@
 F 2 "Resistor_SMD:R_0805_2012Metric" H 1905 7275 50  0001 C CNN
 F 3 "~" H 1905 7275 50  0001 C CNN
+F 4 "C27834" V 1905 7275 50  0001 C CNN "LCSC"
 	1    1905 7275
 	1    0    0    -1
@@
 F 2 "Resistor_SMD:R_0805_2012Metric" H 1780 7275 50  0001 C CNN
 F 3 "~" H 1780 7275 50  0001 C CNN
+F 4 "C27834" V 1780 7275 50  0001 C CNN "LCSC"
 	1    1780 7275
 	1    0    0    -1
@@
 F 2 "Resistor_SMD:R_0805_2012Metric" H 3380 6175 50  0001 C CNN
 F 3 "~" H 3380 6175 50  0001 C CNN
+F 4 "C17561" V 3380 6175 50  0001 C CNN "LCSC"
 	1    3380 6175
 	0    -1   -1   0
@@
 F 2 "Resistor_SMD:R_0805_2012Metric" H 3380 6075 50  0001 C CNN
 F 3 "~" H 3380 6075 50  0001 C CNN
+F 4 "C17561" V 3380 6075 50  0001 C CNN "LCSC"
 	1    3380 6075
 	0    -1   -1   0
@@
 F 2 "Diode_SMD:D_SOD-123" V 8335 2350 50  0001 C CNN
 F 3 "~" V 8335 2350 50  0001 C CNN
+F 4 "C8598" V 8335 2350 50  0001 C CNN "LCSC"
 	1    8335 2350
 	0    -1   -1   0
@@
 F 2 "Diode_SMD:D_SOD-123" V 8315 3000 50  0001 C CNN
 F 3 "~" V 8315 3000 50  0001 C CNN
+F 4 "C8598" V 8315 3000 50  0001 C CNN "LCSC"
 	1    8315 3000
 	0    -1   -1   0
@@
 F 2 "LED_SMD:LED_WS2812B_PLCC4_5.0x5.0mm_P3.2mm" H 10040 3080 50  0001 L TNN
 F 3 "https://cdn-shop.adafruit.com/datasheets/WS2812B.pdf" H 10090 3005 50  0001 L TNN
+F 4 "C114586" H 9990 3380 50  0001 C CNN "LCSC"
 	1    9990 3380
 	1    0    0    -1
@@
 F 2 "LED_SMD:LED_WS2812B_PLCC4_5.0x5.0mm_P3.2mm" H 10040 4180 50  0001 L TNN
 F 3 "https://cdn-shop.adafruit.com/datasheets/WS2812B.pdf" H 10090 4105 50  0001 L TNN
+F 4 "C114586" H 9990 4480 50  0001 C CNN "LCSC"
 	1    9990 4480
 	1    0    0    -1
@@
 Wire Wire Line
 	9690 3930 9690 4480
-Text GLabel 9265 3380 0    50   Input ~ 0
+Text GLabel 9515 3380 0    50   Input ~ 0
 RGBLED
 Text GLabel 4500 3140 2    50   Input ~ 0
 RGBLED
-$Comp
-L Device:R_Small R7
-U 1 1 5F30CAA2
-P 9415 3380
-F 0 "R7" V 9219 3380 50  0000 C CNN
-F 1 "500" V 9310 3380 50  0000 C CNN
-F 2 "Resistor_SMD:R_0805_2012Metric" H 9415 3380 50  0001 C CNN
-F 3 "~" H 9415 3380 50  0001 C CNN
-	1    9415 3380
-	0    1    1    0
-$EndComp
 Wire Wire Line
 	9690 3380 9515 3380
-Wire Wire Line
-	9315 3380 9265 3380
 Wire Wire Line
 	9400 2020 9875 2020
@@
 Text GLabel 9400 1920 2    50   Input ~ 0
 ENC_B
-$Comp
-L Mechanical:MountingHole H1
-U 1 1 5F4872F1
-P 6000 5000
-F 0 "H1" H 6100 5046 50  0000 L CNN
-F 1 "MountingHole" H 6100 4955 50  0000 L CNN
-F 2 "MountingHole:MountingHole_2.2mm_M2" H 6000 5000 50  0001 C CNN
-F 3 "~" H 6000 5000 50  0001 C CNN
-	1    6000 5000
-	1    0    0    -1
-$EndComp
-$Comp
-L Mechanical:MountingHole H2
-U 1 1 5F4893A4
-P 7000 5000
-F 0 "H2" H 7100 5046 50  0000 L CNN
-F 1 "MountingHole" H 7100 4955 50  0000 L CNN
-F 2 "MountingHole:MountingHole_2.2mm_M2" H 7000 5000 50  0001 C CNN
-F 3 "~" H 7000 5000 50  0001 C CNN
-	1    7000 5000
-	1    0    0    -1
-$EndComp
-$Comp
-L Mechanical:MountingHole H3
-U 1 1 5F48C223
-P 6000 5500
-F 0 "H3" H 6100 5546 50  0000 L CNN
-F 1 "MountingHole" H 6100 5455 50  0000 L CNN
-F 2 "MountingHole:MountingHole_2.2mm_M2" H 6000 5500 50  0001 C CNN
-F 3 "~" H 6000 5500 50  0001 C CNN
-	1    6000 5500
-	1    0    0    -1
-$EndComp
-$Comp
-L Mechanical:MountingHole H4
-U 1 1 5F48F252
-P 7000 5500
-F 0 "H4" H 7100 5546 50  0000 L CNN
-F 1 "MountingHole" H 7100 5455 50  0000 L CNN
-F 2 "MountingHole:MountingHole_2.2mm_M2" H 7000 5500 50  0001 C CNN
-F 3 "~" H 7000 5500 50  0001 C CNN
-	1    7000 5500
-	1    0    0    -1
-$EndComp
 Text GLabel 6700 3100 0    50   Input ~ 0
 ROW1
@@
 Text GLabel 4500 2540 2    50   Input ~ 0
 ENC_B
+NoConn ~ 4500 3240
+NoConn ~ 4500 3040
+NoConn ~ 4500 2940
+NoConn ~ 4500 2840
+NoConn ~ 4500 2740
+NoConn ~ 4500 2240
+NoConn ~ 4500 1840
+NoConn ~ 4500 1740
+NoConn ~ 4500 1640
+NoConn ~ 4500 1540
+NoConn ~ 3300 2140
+NoConn ~ 4500 3740
+NoConn ~ 4500 3940
+NoConn ~ 4500 4040
+NoConn ~ 4500 4140
+NoConn ~ 4500 4240
+NoConn ~ 4500 4340
+NoConn ~ 4500 4440
+$Comp
+L Mechanical:MountingHole_Pad H1
+U 1 1 5F28E13C
+P 5020 5920
+F 0 "H1" H 5120 5969 50  0000 L CNN
+F 1 "MountingHole_Pad" H 5120 5878 50  0000 L CNN
+F 2 "MountingHole:MountingHole_2.2mm_M2_Pad" H 5020 5920 50  0001 C CNN
+F 3 "~" H 5020 5920 50  0001 C CNN
+	1    5020 5920
+	1    0    0    -1
+$EndComp
+$Comp
+L Mechanical:MountingHole_Pad H2
+U 1 1 5F28FD97
+P 5390 5930
+F 0 "H2" H 5490 5979 50  0000 L CNN
+F 1 "MountingHole_Pad" H 5490 5888 50  0000 L CNN
+F 2 "MountingHole:MountingHole_2.2mm_M2_Pad" H 5390 5930 50  0001 C CNN
+F 3 "~" H 5390 5930 50  0001 C CNN
+	1    5390 5930
+	1    0    0    -1
+$EndComp
+$Comp
+L Mechanical:MountingHole_Pad H3
+U 1 1 5F292B96
+P 5020 6260
+F 0 "H3" H 5120 6309 50  0000 L CNN
+F 1 "MountingHole_Pad" H 5120 6218 50  0000 L CNN
+F 2 "MountingHole:MountingHole_2.2mm_M2_Pad" H 5020 6260 50  0001 C CNN
+F 3 "~" H 5020 6260 50  0001 C CNN
+	1    5020 6260
+	1    0    0    -1
+$EndComp
+$Comp
+L Mechanical:MountingHole_Pad H4
+U 1 1 5F2956E0
+P 5400 6260
+F 0 "H4" H 5500 6309 50  0000 L CNN
+F 1 "MountingHole_Pad" H 5500 6218 50  0000 L CNN
+F 2 "MountingHole:MountingHole_2.2mm_M2_Pad" H 5400 6260 50  0001 C CNN
+F 3 "~" H 5400 6260 50  0001 C CNN
+	1    5400 6260
+	1    0    0    -1
+$EndComp
 $EndSCHEMATC
